File: pcb/neopixel-network.kicad_pcb (KiCad board)
At the start: 2 copper layers, 73.8 x 73.8 mm, 16 parts, among them U1 LD1117IS50, U2 SN65176BDR, U3 SN65176BDR

Commit message: add updated pcb
Parts:
- added ?: , pcb:neopixel-network-logo, F.Cu at (125.1, 64.7)
- added G***: LOGO, pcb:valley-5x7, F.Cu at (116.5, 102.8)
- added G***: LOGO, pcb:gyttja-14x7, F.Cu at (127.4, 102.8)
- moved REF** 0.64 mm to (93.7, 84.0)
- moved REF** 0.40 mm to (156.0, 84.0)
Other:
- board text added: "+"
- board text added: "-"
- board text added: "DATA"
